File: slushie.kicad_pcb (KiCad board)
At the start: 2 copper layers, 198.1 x 100.8 mm, 184 parts, among them K1 STEP, K10 END, K11 STEP, K12 END, K13 STEP, K14 END, K15 STEP, K16 END, K2 END, K3 STEP, K4 END, K5 STEP, K6 END, K7 STEP, K8 END, K9 STEP, P1 TH0, P2 TH1, P3 TH2, P5 TH3, P6 TH4, P8 TH5, SW1 SPST, SW2 SPST, SW3 SPST, U1 LPCXPRESSO_LPC1769_LPCXPRESSO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, U10 DRV8825, U11 DRV8825, U12 DRV8825, U13 DRV8825, U2 MCP23017, U3 MCP44X1, U4 DRV8825, U5 DRV8825, U6 DRV8825, U7 DRV8825, U8 MCP23017, U9 MCP44X1

Commit message: step wing looking good
Parts:
- removed C20, C24, C29, C33, C37, C41: 0.47µF, SMD_Packages:SMD-0805
- removed C21, C22, C25, C27, C30, C31, C34, C35, C38, C39, C42: 0.1µF, SMD_Packages:SMD-0805
- removed C23, C28, C32, C36, C40: 0.01µF, SMD_Packages:SMD-0805
- removed C26, C43, C44: 1µF, SMD_Packages:SMD-0805
- removed D6: DIODE, Diodes_SMD:D
- removed Ethernet: RJ45-TRANSFO, Connect:RJ45_TRANSFO
- removed I2C: I²C, Pin_Headers:Pin_Header_Angled_1x04
- removed K1, K11, K13, K15, K3, K5, K7, K9: STEP, Pin_Headers:Pin_Header_Angled_1x04
- removed K10, K12, K14, K16, K2, K4, K6, K8: END, Pin_Headers:Pin_Header_Straight_1x03
- removed the Nylon Only at (190.2, 109.7)
- removed the Nylon Only at (90.2, 109.2)
- removed the Nylon Only at (90.2, 17.8)
- removed the Nylon Only at (180.3, 19.1)
- removed the Nylon Only at (39.4, 16.5)
- removed the Nylon Only at (81.3, 16.5)
- removed the Nylon Only at (39.4, 58.4)
- removed the Nylon Only at (80.0, 58.4)
- removed the Nylon Only at (39.4, 67.3)
- removed the Nylon Only at (81.3, 67.3)
- removed the Nylon Only at (81.3, 109.2)
- removed the Nylon Only at (190.2, 67.8)
- removed the Nylon Only at (39.4, 109.2)
- removed the Nylon Only at (229.6, 67.8)
- removed the Nylon Only at (229.6, 109.7)
- removed the Nylon Only at (229.9, 59.7)
- removed the Nylon Only at (229.9, 17.8)
- removed the Nylon Only at (190.5, 17.8)
- removed the Nylon Only at (190.5, 59.7)
- removed the Nylon Only at (181.6, 109.2)
- removed P1: TH0, Pin_Headers:Pin_Header_Straight_1x02
- removed P2: TH1, Pin_Headers:Pin_Header_Straight_1x02
- removed P3: TH2, Pin_Headers:Pin_Header_Straight_1x02
- removed P5: TH3, Pin_Headers:Pin_Header_Straight_1x02
- removed P6: TH4, Pin_Headers:Pin_Header_Straight_1x02
- removed P8: TH5, Pin_Headers:Pin_Header_Straight_1x02
- removed PIN_HEADER_A_2X10 (x8): Val**, Pin_Headers:Pin_Header_Angled_2x10
- removed PWM0-3, PWM3-5: BORN6, Connect:bornier6
- removed R41, R47, R51, R55, R59: 5k6, Resistors_SMD:Resistor_SMD0805_HandSoldering
- removed R42: 100k, Resistors_SMD:Resistor_SMD0805_HandSoldering
- removed R43: 33k, Resistors_SMD:Resistor_SMD0805_HandSoldering
- removed R44, R45, R48, R49, R52, R53, R56, R57: 0.5, Resistors_SMD:Resistor_SMD2512_HandSoldering
- removed R46, R50, R54, R58: 1k, Resistors_SMD:Resistor_SMD0805_HandSoldering
- removed SD CARD: MicroSD, SD:MICRO_SD_HINGE_AMP
- removed SPI: SPI, Pin_Headers:Pin_Header_Angled_1x06
- removed Sym: Symbol_GNU-GPL_CopperTop_Small, Symbols:Symbol_GNU-GPL_CopperTop_Small
- removed U10, U11, U12, U13, U4, U5, U6, U7: DRV8825, Local:TSSOP-28
- removed U3, U9: MCP44X1, Local:TSSOP-20
- removed U8: MCP23017, SMD_Packages:SSOP-28
- removed UART: UART, Pin_Headers:Pin_Header_Angled_1x04
- removed USB: USB-MINI-B, Connect:USB_MINI_B
- added END1: END, Pin_Headers:Pin_Header_Straight_1x03, F.Cu at (58.4, 179.1)
- added END2: END, Pin_Headers:Pin_Header_Straight_1x03, F.Cu at (62.2, 179.1)
- added END3: END, Pin_Headers:Pin_Header_Straight_1x03, F.Cu at (66.0, 179.1)
- added END4: END, Pin_Headers:Pin_Header_Straight_1x03, F.Cu at (69.8, 179.1)
- added END5: END, Pin_Headers:Pin_Header_Straight_1x03, F.Cu at (73.7, 179.1)
- added END6: END, Pin_Headers:Pin_Header_Straight_1x03, F.Cu at (77.5, 179.1)
- added END7: END, Pin_Headers:Pin_Header_Straight_1x03, F.Cu at (81.3, 179.1)
- added END8: END, Pin_Headers:Pin_Header_Straight_1x03, F.Cu at (85.1, 179.1)
- added ETHERNET1: RJ45-TRANSFO, Connect:RJ45_TRANSFO, F.Cu at (108.0, 104.1)
- added I2C1: I²C, Pin_Headers:Pin_Header_Straight_1x04, F.Cu at (68.6, 170.2)
- added L1: 330µH, Inductors:SELF-WE-PD-XXL, F.Cu at (116.8, 167.6)
- added Nylon Only: 3-1mm, Local:MountingHole_3-1mm, F.Cu at (141.0, 88.9)
- added Nylon Only: 3-1mm, Local:MountingHole_3-1mm, F.Cu at (141.0, 180.3)
- added Nylon Only: 3-1mm, Local:MountingHole_3-1mm, F.Cu at (49.5, 180.3)
- added Nylon Only: 3-1mm, Local:MountingHole_3-1mm, F.Cu at (49.5, 88.9)
- added POWER1: BARREL_JACK, Connect:BARREL_JACK, F.Cu at (59.7, 88.9)
- added SD1: MicroSD, SD:MICRO_SD_HINGE_AMP, F.Cu at (118.1, 141.0)
- added SPI1: SPI, Pin_Headers:Pin_Header_Straight_1x06, F.Cu at (87.6, 170.2)
- added TH1: TH, Pin_Headers:Pin_Header_Straight_1x02, F.Cu at (90.2, 180.3)
- added TH2: TH, Pin_Headers:Pin_Header_Straight_1x02, F.Cu at (94.0, 180.3)
- added TH3: TH, Pin_Headers:Pin_Header_Straight_1x02, F.Cu at (97.8, 180.3)
- added TH4: TH, Pin_Headers:Pin_Header_Straight_1x02, F.Cu at (101.6, 180.3)
- added TH5: TH, Pin_Headers:Pin_Header_Straight_1x02, F.Cu at (105.4, 180.3)
- added TH6: TH, Pin_Headers:Pin_Header_Straight_1x02, F.Cu at (109.2, 180.3)
- added UART1: UART, Pin_Headers:Pin_Header_Straight_1x04, F.Cu at (49.5, 97.8)
- added USB1: USB-MINI-B, Connect:USB_MINI_B, F.Cu at (132.1, 88.9)
- added WING1: CONN_4X2, Pin_Headers:Pin_Header_Angled_2x04, F.Cu at (50.8, 109.9)
- added WING2: CONN_4X2, Pin_Headers:Pin_Header_Angled_2x04, F.Cu at (50.8, 160.0)
- added WING3: WINGSTEP, Pin_Headers:Pin_Header_Angled_2x08, F.Cu at (139.7, 109.9)
- added WING4: WINGSTEP, Pin_Headers:Pin_Header_Angled_2x08, F.Cu at (139.7, 160.0)
- added WINGPWR1: WINGPWR, Connect:bornier2, F.Cu at (48.3, 129.5)
- added WINGPWR2: WINGPWR, Connect:bornier2, F.Cu at (48.3, 139.7)
- added WINGPWR3: WINGPWR, Connect:bornier2, F.Cu at (142.2, 129.5)
- added WINGPWR4: WINGPWR, Connect:bornier2, F.Cu at (142.2, 139.7)
- C1, C2: value 10µF -> CP; footprint SMD_Packages:SMD-0805 -> SMD_Packages:SMD-2512_Pol
- C11: value 0.01µF -> 0.1µF
- C12: value 0.47µF -> 0.1µF
- C14, C17, C18: value 0.1µF -> 10µF
- C15, C19: value 0.01µF -> 10µF
- C16: value 0.47µF -> 10µF
- C3: value 10µF -> 4.7nF
- C4: value 10µF -> 1µF
- C5, C6: value 10µF -> 0.1µF
- C7, C9: value 1µF -> 0.1µF
- D1: value LED -> 1N5818; footprint LEDs:LED-0805 -> Diodes_SMD:Diode-Universal-SMB-SMC_Handsoldering
- D5: value DIODE -> LED; footprint Diodes_SMD:D -> LEDs:LED-0805
- R1: value 10k -> 1M
- R11: value 4k7 -> 2k2
- R12, R13, R14, R15: value 4k7 -> 1k
- R16, R17, R18, R19: value 270 -> 1k
- R20, R21, R22, R23: value 10k -> 5k6
- R24: value 100k -> 5k6
- R25: value 33k -> 5k6
- R26, R27: value 0.5 -> 5k6; footprint Resistors_SMD:Resistor_SMD2512_HandSoldering -> Resistors_SMD:Resistor_SMD0805_HandSoldering
- R28, R4, R5: value 1k -> 10k
- R29: value 5k6 -> 10k
- R30: value 0.5 -> 10k; footprint Resistors_SMD:Resistor_SMD2512_HandSoldering -> Resistors_SMD:Resistor_SMD0805_HandSoldering
- R31, R34: value 0.5 -> 1k; footprint Resistors_SMD:Resistor_SMD2512_HandSoldering -> Resistors_SMD:Resistor_SMD0805_HandSoldering
- R33: value 5k6 -> 1k
- R35, R38, R39: value 0.5 -> 4k7; footprint Resistors_SMD:Resistor_SMD2512_HandSoldering -> Resistors_SMD:Resistor_SMD0805_HandSoldering
- R36, R40: value 1k -> 4k7
- R37: value 5k6 -> 4k7
- R6, R7: value 1k -> 270
- R8: value 4k7 -> 270
- R9: value 2k2 -> 270
- U1: value LPCXPRESSO_LPC1769_LPCXPRESSO_LPC1769 -> LM2575; footprint LPCXpresso_boards.mod:LPCXPRESSO_LPC1769 -> SMD_Packages:TO-263-5
- U2: value MCP23017 -> LPC1769 LPCXpresso; footprint SMD_Packages:SSOP-28 -> LPCXpresso_boards.mod:LPCXPRESSO_LPC1769
- moved C15 476.6 mm to (99.1, 186.7)
- moved R31 463.3 mm to (74.9, 158.8), turned to 180 degrees
- moved C9 455.1 mm to (64.8, 196.8), turned to 0 degrees
- moved C17 453.9 mm to (106.7, 186.7)
- moved R32 453.9 mm to (80.0, 158.8), turned to 180 degrees
- moved R25 447.7 mm to (74.9, 193.0), turned to 0 degrees
- moved C14 443.1 mm to (95.2, 186.7), turned to 0 degrees
- moved R24 442.8 mm to (69.8, 193.0), turned to 0 degrees
- moved R39 442.0 mm to (111.8, 175.3)
- moved R40 436.7 mm to (118.1, 175.3), turned to 0 degrees
- moved R33 434.1 mm to (86.4, 158.8), turned to 180 degrees
- moved C16 433.7 mm to (102.9, 186.7)
- moved R30 429.8 mm to (119.4, 125.7)
- moved R38 428.6 mm to (106.7, 175.3)
- moved U2 426.7 mm to (78.7, 55.9), turned to 270 degrees
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Connections:
- C1 pad 1: /TH0 -> +24V
- C1 pad 2: Net-(C1-Pad2) -> GND
- C10 pad 1: +24V -> /END4
- C10 pad 2: Net-(C10-Pad2) -> GND
- C11 pad 1: Net-(C11-Pad1) -> /END5
- C11 pad 2: Net-(C11-Pad2) -> GND
- C12 pad 1: Net-(C12-Pad1) -> /END6
- C13 pad 1: /Stepper0-3/END0 -> /END7
- C14 pad 1: +24V -> /TH0
- C15 pad 1: Net-(C15-Pad1) -> /TH1
- C15 pad 2: Net-(C15-Pad2) -> Net-(C14-Pad2)
- C16 pad 1: Net-(C16-Pad1) -> /TH2
- C16 pad 2: GND -> Net-(C14-Pad2)
- C17 pad 1: /Stepper0-3/END1 -> /TH3
- C17 pad 2: GND -> Net-(C14-Pad2)
- C18 pad 1: +24V -> /TH4
- C18 pad 2: Net-(C18-Pad2) -> Net-(C14-Pad2)
- C19 pad 1: Net-(C19-Pad1) -> /TH5
- C19 pad 2: Net-(C19-Pad2) -> Net-(C14-Pad2)
- C2 pad 1: /TH1 -> +3.3V
- C2 pad 2: Net-(C1-Pad2) -> GND
- C3 pad 1: /TH2 -> Net-(C3-Pad1)
- C3 pad 2: Net-(C1-Pad2) -> GND
- C4 pad 1: /TH3 -> +3.3V
- C4 pad 2: Net-(C1-Pad2) -> GND
- C5 pad 1: /TH4 -> +3.3V
- C5 pad 2: Net-(C1-Pad2) -> GND
- C6 pad 1: /TH5 -> /END0
- C6 pad 2: Net-(C1-Pad2) -> GND
- C7 pad 1: +3.3V -> /END1
- C8 pad 1: +3.3V -> /END2
- C9 pad 1: +3.3V -> /END3
- D1 pad 1: Net-(D1-Pad1) -> GND
- D1 pad 2: GND -> Net-(D1-Pad2)
- D5 pad 2: +5V -> GND
- R1 pad 1: +3.3V -> Net-(C3-Pad1)
- R1 pad 2: /RESET -> GND
- R10 pad 1: /Stepper0-3/SCL -> /SDA
- R11 pad 1: +3.3V -> /SCL
- R11 pad 2: /TH1 -> +3.3V
- R12 pad 2: /TH2 -> Net-(END1-Pad2)
- R13 pad 2: /TH3 -> Net-(END2-Pad2)
- R14 pad 2: /TH4 -> Net-(END3-Pad2)
- R15 pad 2: /TH5 -> Net-(END4-Pad2)
- R16 pad 1: Net-(J2-Pad2) -> +3.3V
- R16 pad 2: /SD -> Net-(END5-Pad2)
- R17 pad 1: Net-(J2-Pad3) -> +3.3V
- R17 pad 2: /MOSI -> Net-(END6-Pad2)
- R18 pad 1: Net-(J2-Pad5) -> +3.3V
- R18 pad 2: /SCK -> Net-(END7-Pad2)
- R19 pad 1: Net-(J2-Pad7) -> +3.3V
- R19 pad 2: /MISO -> Net-(END8-Pad2)
- R2 pad 2: /BOOT -> Net-(R2-Pad2)
- R20 pad 1: +3.3V -> Net-(END1-Pad2)
- R20 pad 2: Net-(J2-Pad2) -> /END0
- R21 pad 1: +3.3V -> Net-(END2-Pad2)
- R21 pad 2: Net-(J2-Pad3) -> /END1
- R22 pad 1: +3.3V -> Net-(END3-Pad2)
- R22 pad 2: Net-(J2-Pad5) -> /END2
- R23 pad 1: +3.3V -> Net-(END4-Pad2)
- R23 pad 2: Net-(J2-Pad7) -> /END3
- R24 pad 1: +3.3V -> Net-(END5-Pad2)
- R24 pad 2: Net-(R24-Pad2) -> /END4
- R25 pad 1: +3.3V -> Net-(END6-Pad2)
- R25 pad 2: Net-(R25-Pad2) -> /END5
- R26 pad 1: Net-(R26-Pad1) -> Net-(END7-Pad2)
- R26 pad 2: GND -> /END6
- R27 pad 1: Net-(R27-Pad1) -> Net-(END8-Pad2)
- R27 pad 2: GND -> /END7
- R28 pad 2: Net-(K2-Pad2) -> /RESET
- R29 pad 1: Net-(K2-Pad2) -> +3.3V
- R29 pad 2: /Stepper0-3/END0 -> /BOOT
- R3 pad 2: /PAUSE -> Net-(R3-Pad2)
- R30 pad 1: Net-(R30-Pad1) -> +3.3V
- R30 pad 2: GND -> /PAUSE
- R31 pad 1: Net-(R31-Pad1) -> /LED1
- R31 pad 2: GND -> Net-(D2-Pad1)
- R32 pad 1: +3.3V -> /LED2
- R32 pad 2: Net-(K4-Pad2) -> Net-(D3-Pad1)
- R33 pad 1: Net-(K4-Pad2) -> /LED3
- R33 pad 2: /Stepper0-3/END1 -> Net-(D4-Pad1)
- R34 pad 1: Net-(R34-Pad1) -> /LED4
- R34 pad 2: GND -> Net-(D5-Pad1)
- R35 pad 1: Net-(R35-Pad1) -> +3.3V
- R35 pad 2: GND -> /TH0
- R36 pad 2: Net-(K6-Pad2) -> /TH1
- R37 pad 1: Net-(K6-Pad2) -> +3.3V
- R37 pad 2: /Stepper0-3/END2 -> /TH2
- R38 pad 1: Net-(R38-Pad1) -> +3.3V
- R38 pad 2: GND -> /TH3
- R39 pad 1: Net-(R39-Pad1) -> +3.3V
- R39 pad 2: GND -> /TH4
- R4 pad 1: /LED1 -> +3.3V
- R4 pad 2: Net-(D1-Pad1) -> Net-(R4-Pad2)
- R40 pad 2: Net-(K8-Pad2) -> /TH5
- R5 pad 1: /LED2 -> +3.3V
- R5 pad 2: Net-(D2-Pad1) -> Net-(R5-Pad2)
- R6 pad 1: /LED3 -> Net-(R2-Pad2)
- R6 pad 2: Net-(D3-Pad1) -> /SD
- R7 pad 1: /LED4 -> Net-(R3-Pad2)
- R7 pad 2: Net-(D4-Pad1) -> /MOSI
- R8 pad 1: +3.3V -> Net-(R4-Pad2)
- R8 pad 2: /TH0 -> /SCK
- R9 pad 1: /Stepper0-3/SDA -> Net-(R5-Pad2)
- R9 pad 2: +3.3V -> /MISO
- U1 pad 1: GND -> +24V
- U1 pad 2: +5V -> Net-(D1-Pad2)
- U1 pad 3: Net-(U1-Pad3) -> GND
- U1 pad 4: /RESET -> +3.3V
- U1 pad 5: /MOSI -> GND
- U2 pad 1: /Stepper0-3/Stepper2/MODE2 -> GND
- U2 pad 10: GND -> /SCL
- U2 pad 11: (no net) -> /DIR7
- U2 pad 12: /Stepper0-3/SCL -> /DIR6
- U2 pad 13: /Stepper0-3/SDA -> /DIR4
- U2 pad 14: (no net) -> /DIR5
- U2 pad 15: GND -> /TH0
- U2 pad 16: +3.3V -> /TH1
- U2 pad 17: +3.3V -> /TH2
- U2 pad 18: +3.3V -> /TH3
- U2 pad 19: Net-(U2-Pad19) -> /TH4
- U2 pad 2: /Stepper0-3/Stepper2/MODE1 -> (no net)
- U2 pad 20: Net-(U2-Pad20) -> /TH5
- U2 pad 21: /Stepper0-3/Stepper0/MODE2 -> /TX
- U2 pad 22: /Stepper0-3/Stepper0/MODE1 -> /RX
- U2 pad 23: /Stepper0-3/Stepper0/MODE0 -> /EN2
- U2 pad 24: /Stepper0-3/Stepper0/DECAY -> /EN3
- U2 pad 25: /Stepper0-3/Stepper1/MODE2 -> /EN4
- U2 pad 26: /Stepper0-3/Stepper1/MODE1 -> /EN5
- U2 pad 27: /Stepper0-3/Stepper1/MODE0 -> /END3
- U2 pad 28: /Stepper0-3/Stepper1/DECAY -> +3.3V
- U2 pad 3: /Stepper0-3/Stepper2/MODE0 -> (no net)
- U2 pad 4: /Stepper0-3/Stepper2/DECAY -> /RESET
- U2 pad 5: /Stepper0-3/Stepper3/MODE2 -> /MOSI
- U2 pad 6: /Stepper0-3/Stepper3/MODE1 -> /MISO
- U2 pad 7: /Stepper0-3/Stepper3/MODE0 -> /SCK
- U2 pad 8: /Stepper0-3/Stepper3/DECAY -> /SD
- U2 pad 9: +3.3V -> /SDA
Routing:
- net +24V: track 0.00 -> 177.9 mm
- net /Stepper4-7/Stepper1/PW: track 91.3 -> 0.00 mm, vias 2 -> 0
- net /Stepper4-7/Stepper0/PW: track 85.3 -> 0.00 mm, vias 2 -> 0
- net GND: track 105.9 -> 40.8 mm, vias 66 -> 2
- net /D-: track 0.00 -> 55.8 mm
- net /D+: track 0.00 -> 50.7 mm
- net /Stepper4-7/Stepper2/PW: track 34.3 -> 0.00 mm, vias 2 -> 0
- net +3.3V: track 68.5 -> 35.0 mm
- net /Stepper0-3/SCL: track 32.3 -> 0.00 mm
- net /Stepper4-7/Stepper3/PW: track 31.1 -> 0.00 mm
- net Net-(C3-Pad1): track 0.00 -> 26.0 mm
- net /Stepper0-3/SDA: track 25.7 -> 0.00 mm
- net /Stepper4-7/Stepper3/DECAY: track 24.4 -> 0.00 mm
- net /Stepper4-7/DIR0: track 24.4 -> 0.00 mm, vias 1 -> 0
- net /Stepper4-7/STEP0: track 24.3 -> 0.00 mm, vias 1 -> 0
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- removed copper zone on F.Cu, net +24V
- removed copper zone on F.Cu, net GND
Other:
- board size 198.1 x 100.8 mm -> 99.1 x 99.1 mm

Commit message: just the spi
Parts:
- moved Nylon Only 213.3 mm to (224.2, 57.8), turned to 180 degrees
- moved Nylon Only 184.8 mm to (224.2, 149.2), turned to 180 degrees
- moved WINGPWR2 181.9 mm to (225.4, 98.4), turned to 90 degrees
- moved WINGPWR1 178.4 mm to (225.4, 108.6), turned to 270 degrees
- moved WING1 175.0 mm to (222.9, 78.1), turned to 270 degrees
- moved WING2 175.0 mm to (222.9, 128.3), turned to 270 degrees
- moved POWER1 159.9 mm to (216.5, 57.8)
- moved R10 157.1 mm to (221.6, 141.5), turned to 90 degrees
- moved I2C1 152.0 mm to (218.3, 144.3), turned to 270 degrees
- moved D2 150.1 mm to (195.6, 78.7), turned to 180 degrees
- moved D3 148.0 mm to (200.7, 78.7), turned to 180 degrees
- moved R31 146.2 mm to (195.6, 76.2), turned to 0 degrees
- moved R32 146.2 mm to (200.7, 76.2), turned to 0 degrees
- moved D4 145.9 mm to (205.7, 78.7), turned to 180 degrees
- moved R11 145.5 mm to (215.3, 143.0), turned to 90 degrees
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Connections:
- ETHERNET1 pad GA: (no net) -> Net-(ETHERNET1-PadGA)
- ETHERNET1 pad GK: (no net) -> Net-(ETHERNET1-PadGK)
- ETHERNET1 pad YA: (no net) -> Net-(ETHERNET1-PadYA)
- ETHERNET1 pad YK: (no net) -> Net-(ETHERNET1-PadYK)
- POWER1 pad 3: (no net) -> Net-(POWER1-Pad3)
- SD1 pad 1: (no net) -> Net-(SD1-Pad1)
- SD1 pad 8: (no net) -> Net-(SD1-Pad8)
- U2 pad 15: /TH0 -> /TH5
- U2 pad 16: /TH1 -> /TH4
- U2 pad 17: /TH2 -> /TH3
- U2 pad 18: /TH3 -> /TH2
- U2 pad 19: /TH4 -> /TH1
- U2 pad 2: (no net) -> Net-(U2-Pad2)
- U2 pad 20: /TH5 -> /TH0
- U2 pad 29: (no net) -> Net-(U2-Pad29)
- U2 pad 3: (no net) -> Net-(U2-Pad3)
- U2 pad 30: (no net) -> Net-(U2-Pad30)
- U2 pad 31: (no net) -> Net-(U2-Pad31)
- USB1 pad 1: (no net) -> Net-(USB1-Pad1)
- USB1 pad 4: (no net) -> Net-(USB1-Pad4)
- WING1 pad 7: (no net) -> Net-(WING1-Pad7)
- WING2 pad 7: (no net) -> Net-(WING2-Pad7)
Routing:
- net +3.3V: track 35.0 -> 366.4 mm
- net /SCL: track 0.00 -> 304.9 mm, vias 0 -> 3
- net /SDA: track 0.00 -> 183.5 mm, vias 0 -> 3
- net GND: track 40.8 -> 188.1 mm, vias 2 -> 19
- net (no net): track 0.00 -> 118.2 mm
- net /TH5: track 0.00 -> 100.6 mm
- net /TH4: track 0.00 -> 93.9 mm
- net /TH3: track 0.00 -> 87.0 mm
- net /TH2: track 0.00 -> 80.7 mm
- net /TH1: track 0.00 -> 74.0 mm
- net /BOOT: track 0.00 -> 73.2 mm, vias 0 -> 1
- net /TH0: track 0.00 -> 69.7 mm
- net /PWM0: track 0.00 -> 68.7 mm
- net /PAUSE: track 0.00 -> 66.6 mm, vias 0 -> 1
- net /RX: track 0.00 -> 62.0 mm
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
Commit message: mainboard
Parts:
- moved SPI1 80.2 mm to (140.3, 142.9)
- moved D1 24.3 mm to (208.9, 106.0), turned to 90 degrees
- moved WING3 21.2 mm to (134.0, 128.3)
- moved C4 14.7 mm to (161.9, 73.0), turned to 0 degrees
- moved C2 12.1 mm to (191.1, 112.4)
- moved R5 11.3 mm to (156.8, 70.5), turned to 180 degrees
- moved L1 11.0 mm to (200.0, 101.0)
- moved R2 10.0 mm to (156.8, 78.1)
- moved R10 10.0 mm to (214.0, 148.0), turned to 270 degrees
- moved C1 9.97 mm to (200.0, 109.9)
- moved U1 9.97 mm to (200.0, 114.9)
- moved C5 8.82 mm to (161.9, 70.5), turned to 0 degrees
- moved R7 7.65 mm to (151.8, 75.6)
- moved R3 6.54 mm to (156.8, 75.6)
- moved R40 6.27 mm to (210.2, 144.1), turned to 180 degrees
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Connections:
- C14 pad 2: Net-(C14-Pad2) -> GND
- C15 pad 2: Net-(C14-Pad2) -> GND
- C16 pad 2: Net-(C14-Pad2) -> GND
- C17 pad 2: Net-(C14-Pad2) -> GND
- C18 pad 2: Net-(C14-Pad2) -> GND
- C19 pad 2: Net-(C14-Pad2) -> GND
- ETHERNET1 pad GA: Net-(ETHERNET1-PadGA) -> (no net)
- ETHERNET1 pad GK: Net-(ETHERNET1-PadGK) -> (no net)
- ETHERNET1 pad YA: Net-(ETHERNET1-PadYA) -> (no net)
- ETHERNET1 pad YK: Net-(ETHERNET1-PadYK) -> (no net)
- I2C1 pad 1: +3.3V -> GND
- I2C1 pad 2: /SDA -> /SCL
- I2C1 pad 3: /SCL -> /SDA
- I2C1 pad 4: GND -> +3.3V
- POWER1 pad 3: Net-(POWER1-Pad3) -> (no net)
- SD1 pad 1: Net-(SD1-Pad1) -> (no net)
- SD1 pad 8: Net-(SD1-Pad8) -> (no net)
- SPI1 pad 1: +3.3V -> GND
- SPI1 pad 2: /LED4 -> /MISO
- SPI1 pad 3: /MOSI -> /SCK
- SPI1 pad 4: /SCK -> /MOSI
- SPI1 pad 5: /MISO -> /LED4
- SPI1 pad 6: GND -> +3.3V
- TH1 pad 1: Net-(C14-Pad2) -> GND
- TH2 pad 1: Net-(C14-Pad2) -> GND
- TH3 pad 1: Net-(C14-Pad2) -> GND
- TH4 pad 1: Net-(C14-Pad2) -> GND
- TH5 pad 1: Net-(C14-Pad2) -> GND
- TH6 pad 1: Net-(C14-Pad2) -> GND
- U2 pad 11: /DIR7 -> /STP4
- U2 pad 12: /DIR6 -> /EN4
- U2 pad 14: /DIR5 -> /STP5
- U2 pad 2: Net-(U2-Pad2) -> (no net)
- U2 pad 23: /EN2 -> /EN6
- U2 pad 24: /EN3 -> /STP7
- U2 pad 25: /EN4 -> /DIR7
- U2 pad 26: /EN5 -> /EN0
- U2 pad 27: /END3 -> /STP1
- U2 pad 29: Net-(U2-Pad29) -> (no net)
- U2 pad 3: Net-(U2-Pad3) -> (no net)
- U2 pad 30: Net-(U2-Pad30) -> (no net)
- U2 pad 31: Net-(U2-Pad31) -> (no net)
- U2 pad 38: /DIR0 -> /LED1
- U2 pad 39: /DIR1 -> /LED2
- U2 pad 40: /DIR2 -> /LED3
- U2 pad 41: /DIR3 -> /LED4
- U2 pad 42: /PWM0 -> /PWM1
- U2 pad 43: /PWM1 -> /PWM2
- U2 pad 44: /PWM2 -> /PWM0
- U2 pad 45: /PWM3 -> /PWM5
- U2 pad 47: /PWM5 -> /PWM3
- U2 pad 48: /EN6 -> /END4
- U2 pad 49: /EN7 -> /END5
- U2 pad 50: /END0 -> /END6
- U2 pad 52: /END2 -> /END7
- U2 pad 55: /END1 -> /DIR6
- U2 pad 56: /EN1 -> /EN7
- U2 pad 57: /EN0 -> /STP0
- U2 pad 58: /END7 -> /DIR0
- U2 pad 59: /END6 -> /STP6
- U2 pad 60: /END5 -> /DIR1
- U2 pad 61: /END4 -> /EN1
- U2 pad 62: /STP7 -> /DIR5
- U2 pad 63: /STP6 -> /EN2
- U2 pad 64: /STP5 -> /STP2
- U2 pad 65: /STP4 -> /EN5
- U2 pad 67: /STP2 -> /DIR2
- U2 pad 68: /STP1 -> /END3
- U2 pad 69: /STP0 -> /DIR3
- U2 pad 70: /LED4 -> /EN3
- U2 pad 71: /LED3 -> /END2
- U2 pad 72: /LED2 -> /END0
- U2 pad 73: /LED1 -> /END1
- UART1 pad 1: +3.3V -> GND
- UART1 pad 2: /TX -> /RX
- UART1 pad 3: /RX -> /TX
- UART1 pad 4: GND -> +3.3V
- USB1 pad 1: Net-(USB1-Pad1) -> (no net)
- USB1 pad 4: Net-(USB1-Pad4) -> (no net)
- WING1 pad 7: Net-(WING1-Pad7) -> (no net)
- WING2 pad 7: Net-(WING2-Pad7) -> (no net)
Routing:
- net GND: track 188.1 -> 534.2 mm, vias 19 -> 53
- net +3.3V: track 366.4 -> 613.5 mm, vias 0 -> 6
- net (no net): track 118.2 -> 0.00 mm
- net /SDA: track 183.5 -> 276.1 mm, vias 3 -> 1
- net /MOSI: track 10.8 -> 97.5 mm, vias 0 -> 1
- net +24V: track 146.1 -> 225.0 mm
- net /MISO: track 3.14 -> 81.5 mm, vias 0 -> 1
- net /SCK: track 4.48 -> 82.1 mm, vias 0 -> 1
- net /LED4: track 54.8 -> 126.6 mm, vias 0 -> 1
- net /DIR5: track 13.0 -> 58.3 mm
- net /EN7: track 0.00 -> 43.0 mm
- net /EN6: track 0.00 -> 41.1 mm
- net /PWM4: track 50.4 -> 88.2 mm
- net /PWM5: track 49.7 -> 86.7 mm
- net /END5: track 1.90 -> 36.7 mm, vias 0 -> 1
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- added copper zone on F.Cu, net GND
- added copper zone on F.Cu, net Net-(C3-Pad1)
Other:
- board text added: "+"
- board text added: "-"
- board text added: "24V"
- board text added: "3.3V"
- board text added: "BOOTLOAD"
- board text added: "CS"
- board text added: "END1"
- board text added: "END2"
- board text added: "END3"
- board text added: "END4"
- board text added: "END5"
- board text added: "END6"
- board text added: "END7"
- board text added: "END8"
- board text added: "I²C"
- board text added: "LED1"
- board text added: "LED2"
- board text added: "LED3"
- board text added: "LED4"
- board text added: "LPC1769 LPCXpresso"
- board text added: "MISO"
- board text added: "MOSi"
- board text added: "PAUSE"
- board text added: "R31:4"
- board text added: "RESET"
- board text added: "RX"
- board text added: "SCK"
- board text added: "SCL"
- board text added: "SDA"
- board text added: "SPI"
- board text added: "TH1"
- board text added: "TH2"
- board text added: "TH3"
- board text added: "TH4"
- board text added: "TH5"
- board text added: "TH6"
- board text added: "TX"
- board text added: "v0.0.1 Slushie ©2014 b@Zi.iS CERN OHL v.1.2"
